Commit message: added extra support for the robot

File: palletizing_robot_description/urdf/palletizing_robot.urdf.xacro (robot description, xacro)
@@ -2,4 +2,33 @@
 <robot xmlns:xacro="http://wiki.ros.org/xacro" name="pr">
     <link name="world" />
+    <material name="grey">
+        <color rgba="0.5 0.5 0.5 1"/>
+    </material>
+    <!-- Support -->
+    <link name="support_link">
+        <visual>
+            <origin rpy="0.0 0.0 0" xyz="0 0 0.25"/>
+            <geometry>
+                <cylinder length="0.5" radius="0.1"/>
+            </geometry>
+            <material name="grey"/>
+        </visual>
+        <collision>
+            <origin rpy="0.0 0.0 0" xyz="0 0 0.25"/>
+            <geometry>
+                <cylinder length="0.5" radius="0.1"/>
+            </geometry>
+        </collision>
+        <inertial>
+            <origin rpy="0 0 0" xyz="0 0 0"/>
+            <mass value="20"/>
+            <inertia ixx="0.46" ixy="0.0" ixz="0.0" iyy="0.46" iyz="0.0" izz="0.1"/>
+        </inertial>
+    </link>
+    <joint name="support_joint" type="fixed">
+      <origin rpy="0 0 0" xyz="0 0 0"/>
+      <parent link="world" />
+      <child link="support_link" />
+    </joint>
     <!-- Robot -->
     <xacro:include filename="$(find ur_description)/urdf/ur_macro.xacro"/>
@@ -7,6 +36,6 @@
         name="pr"
         tf_prefix=""
-        parent="world"
-        joint_limits_parameters_file="$(find ur_description)/config/ur10e/joint_limits.yaml"
+        parent="support_link"
+        joint_limits_parameters_file="$(find palletizing_robot_description)/config/joint_limits.yaml"
         kinematics_parameters_file="$(find ur_description)/config/ur10e/default_kinematics.yaml"
         physical_parameters_file="$(find ur_description)/config/ur10e/physical_parameters.yaml"
@@ -15,5 +44,5 @@
         sim_gazebo="true"
         >
-        <origin xyz="0 0 0" rpy="0 0 0" />
+        <origin xyz="0 0 0.5" rpy="0 0 0" />
     </xacro:ur_robot>
     <!-- Gripper -->
@@ -21,4 +50,7 @@
     <xacro:gripper parent="wrist_3_link" />
     <gazebo reference="world">
+    </gazebo>
+    <gazebo reference="support_link">
+       <material>Gazebo/Grey</material>
     </gazebo>
     <gazebo>
